Commit message: 更改urdf mesh路径

File: legged_lab/assets/tiangong2plus/urdf/tiangong2_plus_urdf.urdf (robot description, URDF)
Before this commit: robot tiangong2_plus_urdf, 26 links, 25 joints
Links:
- link ankle_pitch_l_link: geometry collision mesh filename=../meshes/ankle_pitch_l_link.STL; visual mesh filename=../meshes/ankle_pitch_l_link.STL
- link ankle_pitch_r_link: geometry collision mesh filename=../meshes/ankle_pitch_r_link.STL; visual mesh filename=../meshes/ankle_pitch_r_link.STL
- link ankle_roll_l_link: geometry collision mesh filename=../meshes/ankle_roll_l_link.STL; visual mesh filename=../meshes/ankle_roll_l_link.STL
- link ankle_roll_r_link: geometry collision mesh filename=../meshes/ankle_roll_r_link.STL; visual mesh filename=../meshes/ankle_roll_r_link.STL
- link camera_body_back_link: geometry collision mesh filename=../meshes/camera_body_back_link.STL; visual mesh filename=../meshes/camera_body_back_link.STL
- link camera_body_front_link: geometry collision mesh filename=../meshes/camera_body_front_link.STL; visual mesh filename=../meshes/camera_body_front_link.STL
- link camera_head_link: geometry collision mesh filename=../meshes/camera_head_link.STL; visual mesh filename=../meshes/camera_head_link.STL
- link elbow_pitch_l_link: geometry collision mesh filename=../meshes/elbow_pitch_l_link.STL; visual mesh filename=../meshes/elbow_pitch_l_link.STL
- link elbow_pitch_r_link: geometry collision mesh filename=../meshes/elbow_pitch_r_link.STL; visual mesh filename=../meshes/elbow_pitch_r_link.STL
- link hip_pitch_l_link: geometry collision mesh filename=../meshes/hip_pitch_l_link.STL; visual mesh filename=../meshes/hip_pitch_l_link.STL
- link hip_pitch_r_link: geometry collision mesh filename=../meshes/hip_pitch_r_link.STL; visual mesh filename=../meshes/hip_pitch_r_link.STL
- link hip_roll_l_link: geometry collision mesh filename=../meshes/hip_roll_l_link.STL; visual mesh filename=../meshes/hip_roll_l_link.STL
- link hip_roll_r_link: geometry collision mesh filename=../meshes/hip_roll_r_link.STL; visual mesh filename=../meshes/hip_roll_r_link.STL
- link hip_yaw_l_link: geometry collision mesh filename=../meshes/hip_yaw_l_link.STL; visual mesh filename=../meshes/hip_yaw_l_link.STL
- link hip_yaw_r_link: geometry collision mesh filename=../meshes/hip_yaw_r_link.STL; visual mesh filename=../meshes/hip_yaw_r_link.STL
- link imu_link: geometry collision mesh filename=../meshes/imu_link.STL; visual mesh filename=../meshes/imu_link.STL
- link knee_pitch_l_link: geometry collision mesh filename=../meshes/knee_pitch_l_link.STL; visual mesh filename=../meshes/knee_pitch_l_link.STL
- link knee_pitch_r_link: geometry collision mesh filename=../meshes/knee_pitch_r_link.STL; visual mesh filename=../meshes/knee_pitch_r_link.STL
- link pelvis: geometry collision mesh filename=../meshes/pelvis.STL; visual mesh filename=../meshes/pelvis.STL
- link shoulder_pitch_l_link: geometry collision mesh filename=../meshes/shoulder_pitch_l_link.STL; visual mesh filename=../meshes/shoulder_pitch_l_link.STL
- link shoulder_pitch_r_link: geometry collision mesh filename=../meshes/shoulder_pitch_r_link.STL; visual mesh filename=../meshes/shoulder_pitch_r_link.STL
- link shoulder_roll_l_link: geometry collision mesh filename=../meshes/shoulder_roll_l_link.STL; visual mesh filename=../meshes/shoulder_roll_l_link.STL
- link shoulder_roll_r_link: geometry collision mesh filename=../meshes/shoulder_roll_r_link.STL; visual mesh filename=../meshes/shoulder_roll_r_link.STL
- link shoulder_yaw_l_link: geometry collision mesh filename=../meshes/shoulder_yaw_l_link.STL; visual mesh filename=../meshes/shoulder_yaw_l_link.STL
- link shoulder_yaw_r_link: geometry collision mesh filename=../meshes/shoulder_yaw_r_link.STL; visual mesh filename=../meshes/shoulder_yaw_r_link.STL
- link waist_yaw_link: geometry collision mesh filename=../meshes/waist_yaw_link.STL; visual mesh filename=../meshes/waist_yaw_link.STL
